File: pcb/modulo_SIM7000G/_autosave-modulo_SIM7000G.sch (KiCad schematic (older format))
At the start: 58 parts, among them J1 Conn_01x04, J2 115Q-BCA0, J3 CONECTOR SERIAL, J4 Conn_01x02, J5 DCJ200-10-A-XX-X_REVA, Q1 NTE4153NT1G, Q2 NTE4153NT1G, Q3 NTE4153NT1G, U1 SIM7000G, U2 SN74LV1T34DCKR, U3 SN74LV1T34DCKR, U4 SN74LV1T34DCKR, U5 SN74LV1T34DCKR, U6 SN74LV1T34DCKR, U7 MIC29302WU, U8 LM1117-3.3

Commit message: Acomodando archivos y carpetas del repo
Parts:
- J2: symbol 115Q-BCA0:115Q-BCA0 -> modulo_SIM7000G-rescue:115Q-BCA0-115Q-BCA0
Changed lines of the file:
@@
 	4200 7700 5600 7700
 $Comp
-L 115Q-BCA0:115Q-BCA0 J2
+L modulo_SIM7000G-rescue:115Q-BCA0-115Q-BCA0 J2
 U 1 1 614DFEAF
 P 4200 6300
