File: pcb/modulo_SIM7000G/modulo_SIM7000G.sch (KiCad schematic (older format))
At the start: 19 parts

Commit message: avances en el esquematico(casi terminado) consultar detalles sobre como poner referencias a USB33, VBAT, VEXT, ect
Parts:
- removed C? (x4): C, symbol Device:C
- removed D?: LED, symbol Device:LED
- removed R?: R, symbol Device:R
- removed U? (x3): SN74LV1T34DCKR, symbol SN74LV1T34DCKR:SN74LV1T34DCKR
- added AE?: GNSS, symbol Device:Antenna
- added AE?: CELULAR, symbol Device:Antenna
- added C1, C? (x3): CP_Small, symbol Device:CP_Small
- added C5, C6, C7, C8, C9, C? (x6): C, symbol Device:C
- added J1: Conn_01x04, symbol Connector_Generic:Conn_01x04
- added J2: SIM_Card, symbol Connector:SIM_Card
- added L?: L, symbol Device:L
- added R1, R2, R? (x5): R, symbol Device:R
- added R3, R4, R5: 22, symbol Device:R
- added U2, U3, U4, U5, U6: SN74LV1T34DCKR, symbol SN74LV1T34DCKR:SN74LV1T34DCKR
- added U?: MIC29302WU, Package_TO_SOT_SMD:TO-263-5_TabPin3, symbol Regulator_Linear:MIC29302WU
- gave numbers to parts that had none: 10
Connections:
- net labels added: +BATT, GND, MDM_PWRKEY, MDM_RESET
- wire segments 92 -> 181
Other:
- note added: "CONECTOR USB"
- note added: "INTERFAZ SERIAL"
- note added: "LECTOR SIMCARD"
- moved on the sheet: C2, C3, C4, D1, Q1, Q2, Q3, R6, R7, U1

Commit message: mejora en el esquematico
Connections:
- net labels removed: GNDD, GNDREF
Other:
- note added: "ANTENAS"
- note added: "REGULADOR DE TENSION"
- moved on the sheet: AE?, C1, C2, C3, C4, C5, C6, C7, C8, C9, C?, L?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

Commit message: avance en el esquematico, se posiciono todos los componentes, solo falta agregar VBAT, V5EXT y otras referencia de tension donde corresponda
Parts:
- removed C7: C, symbol Device:C
- added C18, C19, C20: C, symbol Device:C
- added D2: LED, symbol Device:LED
- added D3: DIODE, symbol Simulation_SPICE:DIODE
- added J3: CONECTOR SERIAL, symbol Connector_Generic:Conn_01x04
- added J4: Conn_01x02, symbol Connector_Generic:Conn_01x02
- added R13: R, symbol Device:R
- added U8: LM1117-2.5, symbol Regulator_Linear:LM1117-2.5
- gave numbers to parts that had none: 18
Connections:
- net labels added: +3.3V, +5V, VEE
- net labels removed: MDM_PWRKEY, MDM_RESET
- wire segments 181 -> 209
Other:
- note added: "FUENTE USB (3.3V)"
- note added: "INTERFAZ UART"
- note added: "LED DE ESTADOS\n"
- note added: "NETLIGHT"
- note added: "POWER Y RESET"
- note removed: "INTERFAZ SERIAL"
- moved on the sheet: D1, J1, Q1, Q2, Q3, R1, R2, R6, R7, U6

Commit message: se agregaron valores a componentes
Parts:
- removed C12: CP_Small, symbol Device:CP_Small
- added C5: 100nF, symbol Device:C
- added U9: LM1117-2.5, symbol Regulator_Linear:LM1117-2.5
- C1, C11: value CP_Small -> 100uFx16V
- C10, C2: value C -> 1uF
- C13, C14, C15, C16, C17, C4: value C -> 47pF
- C18, C3: value C -> 100nF
- C19, C20: value C -> 10uF
- C7: value CP_Small -> 470uFx16V
- L1: value L -> 47nH
- R1, R2, R6, R8: value R -> 10K
- R10: value R -> 47K
- R11: value R -> 470K
- R12: value R -> 10
- R13, R7: value R -> 330
- R9: value R -> 100K
- renumbered C5 to 100nF1, C6 to 100nF2, C8 to 100nF3, C9 to 100nF4
Connections:
- net labels added: +3V3
- wire segments 209 -> 212
- no-connect marks 0 -> 15
Other:
- moved on the sheet: 100nF1, 100nF2, 100nF3, 100nF4, C11, C17, C18, D1, D2, J3, Q3, R11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

Commit message: Modificaciones en el esquematico, se agrego un conector lector de sim modelo 115Q-BCA0
Parts:
- removed 100nF1, 100nF2, 100nF3, 100nF4: C, symbol Device:C
- removed J2: SIM_Card, symbol Connector:SIM_Card
- removed R8: 10K, symbol Device:R
- removed U8, U9: LM1117-2.5, symbol Regulator_Linear:LM1117-2.5
- added C12, C21, C22, C6, C8, C9: 100nF, Capacitor_SMD:C_0805_2012Metric_Pad1.18x1.45mm_HandSolder, symbol Device:C
- added J2: 115Q-BCA0, 115Q-BCA0:115QBCA0, symbol 115Q-BCA0:115Q-BCA0
- added J5: DCJ200-10-A-XX-X_REVA, Connector_BarrelJack:BarrelJack_CUI_PJ-063AH_Horizontal, symbol DCJ200-10-A-XX-X_REVA:DCJ200-10-A-XX-X_REVA
- added U8: LM1117-3.3, Package_TO_SOT_SMD:SOT-223, symbol Regulator_Linear:LM1117-3.3
- C1, C11: footprint (none) -> Capacitor_SMD:CP_Elec_6.3x9.9
- C10, C13, C17, C18, C19, C2, C20, C3, C4, C5: footprint (none) -> Capacitor_SMD:C_0805_2012Metric_Pad1.18x1.45mm_HandSolder
- C14, C15, C16: value 47pF -> C; footprint (none) -> Capacitor_SMD:C_0805_2012Metric_Pad1.18x1.45mm_HandSolder
- C7: footprint (none) -> Capacitor_SMD:CP_Elec_8x10
- D1, D2: footprint (none) -> LED_SMD:LED_0805_2012Metric
- D3: footprint (none) -> Diode_SMD:D_0805_2012Metric_Pad1.15x1.40mm_HandSolder
- J1: footprint (none) -> Connector_PinHeader_2.00mm:PinHeader_1x04_P2.00mm_Vertical
- J3: footprint (none) -> Connector:FanPinHeader_1x04_P2.54mm_Vertical
- J4: footprint (none) -> Connector_PinHeader_2.00mm:PinHeader_1x02_P2.00mm_Vertical
- L1: footprint (none) -> Inductor_SMD:L_0805_2012Metric
- Q1, Q2, Q3: footprint SOTFL50P160X80-3N -> Package_TO_SOT_SMD:SOT-416
- R1, R10, R11, R12, R13, R2, R3, R4, R5, R6, R7, R9: footprint (none) -> Resistor_SMD:R_0805_2012Metric
- U1: footprint (none) -> RF_GSM:SIM7000
- U2, U3, U4, U5, U6: footprint (none) -> Package_TO_SOT_SMD:SOT-23-5
Connections:
- net labels added: +5VEXT, USB33, VBAT, VDDX
- net labels removed: +3.3V, +3V3, +5V, +BATT, VDD, VEE
- wire segments 212 -> 265
- no-connect marks 15 -> 19
Other:
- moved on the sheet: C1, C10, C11, C18, C19, C2, C3, C4, C5, C7, D3, R10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

Commit message: Acomodando archivos y carpetas del repo
Parts:
- added FID1, FID2: Fiducial, Fiducial:Fiducial_1mm_Mask2mm, symbol Mechanical:Fiducial
- C14, C15, C16: value C -> 47pF
Changed lines of the file:
@@
 U 1 1 614D3DBD
 P -6200 -4000
-F 0 "U1" H 4300 -11150 50  0000 C CNN
+F 0 "U1" H -6150 -3950 50  0000 C CNN
 F 1 "SIM7000G" H 4350 -11060 50  0000 C CNN
 F 2 "RF_GSM:SIM7000" H 3500 -11200 50  0001 C CNN
@@
 P 5450 5750
 F 0 "C14" H 5450 5650 50  0000 L CNN
-F 1 "C" H 5450 5550 50  0000 L CNN
+F 1 "47pF" H 5450 5550 50  0000 L CNN
 F 2 "Capacitor_SMD:C_0805_2012Metric_Pad1.18x1.45mm_HandSolder" H 5488 5600 50  0001 C CNN
 F 3 "~" H 5450 5750 50  0001 C CNN
@@
 P 5650 5750
 F 0 "C15" H 5650 5650 50  0000 L CNN
-F 1 "C" H 5650 5550 50  0000 L CNN
+F 1 "47pF" H 5650 5550 50  0000 L CNN
 F 2 "Capacitor_SMD:C_0805_2012Metric_Pad1.18x1.45mm_HandSolder" H 5688 5600 50  0001 C CNN
 F 3 "~" H 5650 5750 50  0001 C CNN
@@
 P 5850 5750
 F 0 "C16" H 5850 5650 50  0000 L CNN
-F 1 "C" H 5850 5550 50  0000 L CNN
+F 1 "47pF" H 5850 5550 50  0000 L CNN
 F 2 "Capacitor_SMD:C_0805_2012Metric_Pad1.18x1.45mm_HandSolder" H 5888 5600 50  0001 C CNN
 F 3 "~" H 5850 5750 50  0001 C CNN
@@
 	1    0    0    -1
 $EndComp
+$Comp
+L Mechanical:Fiducial FID1
+U 1 1 61548E6D
+P 7650 6250
+F 0 "FID1" H 7735 6296 50  0000 L CNN
+F 1 "Fiducial" H 7735 6205 50  0000 L CNN
+F 2 "Fiducial:Fiducial_1mm_Mask2mm" H 7650 6250 50  0001 C CNN
+F 3 "~" H 7650 6250 50  0001 C CNN
+	1    7650 6250
+	1    0    0    -1
+$EndComp
+$Comp
+L Mechanical:Fiducial FID2
+U 1 1 6154C0F9
+P 8150 6250
+F 0 "FID2" H 8235 6296 50  0000 L CNN
+F 1 "Fiducial" H 8235 6205 50  0000 L CNN
+F 2 "Fiducial:Fiducial_1mm_Mask2mm" H 8150 6250 50  0001 C CNN
+F 3 "~" H 8150 6250 50  0001 C CNN
+	1    8150 6250
+	1    0    0    -1
+$EndComp

Commit message: Se agrego connectores de antenas
Parts:
- removed AE1: GNSS, symbol Device:Antenna
- removed AE2: CELULAR, symbol Device:Antenna
- added J6, J7: 1661, conn_ufl:1661, symbol conn_ufl:1661
- J2: symbol 115Q-BCA0:115Q-BCA0 -> modulo_SIM7000G-rescue:115Q-BCA0-115Q-BCA0
Connections:
- net at U1.60 (RF_ANT): now also J7.1
- net at C17.1, L1.2: now also J6.1
Changed lines of the file:
@@
 Wire Wire Line
 	5400 2200 5400 2100
-Connection ~ 6000 1600
-Wire Wire Line
-	6000 1350 6000 1600
 Wire Wire Line
 	5850 1600 6000 1600
@@
 	1    0    0    -1
 $EndComp
-$Comp
-L Device:Antenna AE2
-U 1 1 61743083
-P 6400 1150
-F 0 "AE2" H 6480 1139 50  0000 L CNN
-F 1 "CELULAR" H 6480 1048 50  0000 L CNN
-F 2 "" H 6400 1150 50  0001 C CNN
-F 3 "~" H 6400 1150 50  0001 C CNN
-	1    6400 1150
-	1    0    0    -1
-$EndComp
-$Comp
-L Device:Antenna AE1
-U 1 1 617425D0
-P 6000 1150
-F 0 "AE1" H 6080 1139 50  0000 L CNN
-F 1 "GNSS" H 6080 1048 50  0000 L CNN
-F 2 "" H 6000 1150 50  0001 C CNN
-F 3 "~" H 6000 1150 50  0001 C CNN
-	1    6000 1150
-	1    0    0    -1
-$EndComp
 Wire Wire Line
 	4100 2900 6000 2900
 Wire Wire Line
 	6000 2100 6000 2900
-Wire Wire Line
-	6400 1350 6400 3100
-Wire Wire Line
-	4650 3100 6400 3100
 Wire Wire Line
 	3850 2100 3850 2300
@@
 	4200 7700 5600 7700
 $Comp
-L 115Q-BCA0:115Q-BCA0 J2
+L modulo_SIM7000G-rescue:115Q-BCA0-115Q-BCA0 J2
 U 1 1 614DFEAF
 P 4200 6300
@@
 	1    0    0    -1
 $EndComp
+$Comp
+L conn_ufl:1661 J7
+U 1 1 615BD618
+P 6450 1600
+F 0 "J7" V 6745 1472 60  0000 R CNN
+F 1 "1661" V 6639 1472 60  0000 R CNN
+F 2 "conn_ufl:1661" H 6850 1540 60  0001 C CNN
+F 3 "" H 6450 1600 60  0000 C CNN
+	1    6450 1600
+	0    -1   -1   0
+$EndComp
+$Comp
+L conn_ufl:1661 J6
+U 1 1 6160E28F
+P 6000 1600
+F 0 "J6" V 6295 1472 60  0000 R CNN
+F 1 "1661" V 6189 1472 60  0000 R CNN
+F 2 "conn_ufl:1661" H 6400 1540 60  0001 C CNN
+F 3 "" H 6000 1600 60  0000 C CNN
+	1    6000 1600
+	0    -1   -1   0
+$EndComp
+Connection ~ 6000 1600
+Wire Wire Line
+	6450 1600 6450 3100
+Wire Wire Line
+	4650 3100 6450 3100
 $EndSCHEMATC

Commit message: Se generaron los archivos de asignacion de huellas y figuras 3d
Parts:
- J3: value CONECTOR SERIAL -> INTERFAZ SERIAL
- J5: symbol DCJ200-10-A-XX-X_REVA:DCJ200-10-A-XX-X_REVA -> modulo_SIM7000G-rescue:DCJ200-10-A-XX-X_REVA-DCJ200-10-A-XX-X_REVA
- J6, J7: symbol conn_ufl:1661 -> modulo_SIM7000G-rescue:1661-conn_ufl
Other:
- note added: "LED DE ESTADO\n"
- note added: "REGULADOR USB (3.3V)"
- note removed: "FUENTE USB (3.3V)"
- note removed: "LED DE ESTADOS\n"
Changed lines of the file:
@@
 encoding utf-8
 Sheet 1 1
-Title "Modulo de comunicacion basado en SIM7000G"
+Title "Replica modulo de comunicacion basado en SIM7000G"
 Date "2021-09-08"
 Rev "Diego Brengi "
 Comp "FIUBA"
-Comment1 "Descripcion: Modulo de comunicacion basado en SIM7000G(GPRS,4G Y GNSS)"
+Comment1 "Descripcion: Replica modulo de comunicacion basado en SIM7000G(GPRS,4G Y GNSS)"
 Comment2 "Autor: German Gabriel Velardez"
 Comment3 ""
@@
 P 10750 2700
 F 0 "J3" H 10830 2692 50  0000 L CNN
-F 1 "CONECTOR SERIAL" H 10550 2350 50  0000 L CNN
+F 1 "INTERFAZ SERIAL" H 10550 2350 50  0000 L CNN
 F 2 "Connector:FanPinHeader_1x04_P2.54mm_Vertical" H 10750 2700 50  0001 C CNN
 F 3 "~" H 10750 2700 50  0001 C CNN
@@
 	7450 4200 7450 4750
 Text Notes 10450 4750 0    50   ~ 0
-LED DE ESTADOS\n
+LED DE ESTADO\n
 Wire Wire Line
 	3000 4100 3000 7550
@@
 	550  6950 2300 6950
 Text Notes 550  5900 0    50   ~ 0
-FUENTE USB (3.3V)
+REGULADOR USB (3.3V)
 Text Notes 9000 5350 0    50   ~ 0
 NETLIGHT
@@
 	3550 1500 3650 1500
 $Comp
-L DCJ200-10-A-XX-X_REVA:DCJ200-10-A-XX-X_REVA J5
+L modulo_SIM7000G-rescue:DCJ200-10-A-XX-X_REVA-DCJ200-10-A-XX-X_REVA J5
 U 1 1 614B53F2
 P 3250 1300
@@
 $EndComp
 $Comp
-L conn_ufl:1661 J7
+L modulo_SIM7000G-rescue:1661-conn_ufl J7
 U 1 1 615BD618
 P 6450 1600
@@
 $EndComp
 $Comp
-L conn_ufl:1661 J6
+L modulo_SIM7000G-rescue:1661-conn_ufl J6
 U 1 1 6160E28F
 P 6000 1600
