File: pcb/modulo_SIM7000G/modulo_SIM7000G.sch (KiCad schematic (older format))
At the start: 58 parts, among them J1 Conector Serial, J2 115Q-BCA0, J5 Jack-DC, J6 1661, J7 1661, Q1 NTE4153NT1G, Q2 NTE4153NT1G, Q3 NTE4153NT1G, U1 SIM7000G, U2 SN74LV1T34DCKR, U3 SN74LV1T34DCKR, U4 SN74LV1T34DCKR, U5 SN74LV1T34DCKR, U6 SN74LV1T34DCKR, U7 MIC29302WU, U8 LM1117-3.3

Commit message: termine, falta los modelos 3d de los conectores.
Parts:
- removed J6, J7: 1661, Connector_Coaxial:U.FL_Molex_MCRF_73412-0110_Vertical, symbol modulo_SIM7000G-rescue:1661-conn_ufl-modulo_SIM7000G-rescue
- added FID3: Fiducial, Fiducial:Fiducial_1mm_Mask2mm, symbol Mechanical:Fiducial
- added J3: RF ANT, Connector_Coaxial:SMA_Amphenol_132203-12_Horizontal, symbol Connector:Conn_Coaxial
- added J4: GNSS ANT, Connector_Coaxial:SMA_Amphenol_132203-12_Horizontal, symbol Connector:Conn_Coaxial
Connections:
- net GND: now also J3.2 (Ext), J4.2 (Ext)
- net at U1.60 (RF_ANT): now also J3.1 (In)
- net at C17.1, L1.2: now also J4.1 (In)
Other:
- note added: "50 Ohms"
- moved on the sheet: FID1, FID2
Changed lines of the file:
@@
 L Mechanical:Fiducial FID1
 U 1 1 61548E6D
-P 8900 1300
-F 0 "FID1" H 8985 1346 50  0000 L CNN
-F 1 "Fiducial" H 8985 1255 50  0000 L CNN
-F 2 "Fiducial:Fiducial_1mm_Mask2mm" H 8900 1300 50  0001 C CNN
-F 3 "~" H 8900 1300 50  0001 C CNN
-	1    8900 1300
+P 8650 1300
+F 0 "FID1" H 8735 1346 50  0000 L CNN
+F 1 "Fiducial" H 8735 1255 50  0000 L CNN
+F 2 "Fiducial:Fiducial_1mm_Mask2mm" H 8650 1300 50  0001 C CNN
+F 3 "~" H 8650 1300 50  0001 C CNN
+	1    8650 1300
 	1    0    0    -1
 $EndComp
@@
 L Mechanical:Fiducial FID2
 U 1 1 6154C0F9
-P 9550 1300
-F 0 "FID2" H 9635 1346 50  0000 L CNN
-F 1 "Fiducial" H 9635 1255 50  0000 L CNN
-F 2 "Fiducial:Fiducial_1mm_Mask2mm" H 9550 1300 50  0001 C CNN
-F 3 "~" H 9550 1300 50  0001 C CNN
-	1    9550 1300
+P 9300 1300
+F 0 "FID2" H 9385 1346 50  0000 L CNN
+F 1 "Fiducial" H 9385 1255 50  0000 L CNN
+F 2 "Fiducial:Fiducial_1mm_Mask2mm" H 9300 1300 50  0001 C CNN
+F 3 "~" H 9300 1300 50  0001 C CNN
+	1    9300 1300
 	1    0    0    -1
 $EndComp
@@
 CONECTORES DE ANTENAS
 Wire Notes Line
-	7900 700  6350 700
-Wire Notes Line
 	6350 700  6350 2600
 Wire Notes Line
-	7900 2600 7900 700
-Wire Notes Line
-	6350 2600 7900 2600
+	8100 2600 8100 700
 Wire Wire Line
 	7100 2100 7100 2700
-$Comp
-L modulo_SIM7000G-rescue:1661-conn_ufl-modulo_SIM7000G-rescue J7
-U 1 1 615BD618
-P 7550 1600
-F 0 "J7" V 7845 1472 60  0000 R CNN
-F 1 "1661" V 7739 1472 60  0000 R CNN
-F 2 "Connector_Coaxial:U.FL_Molex_MCRF_73412-0110_Vertical" H 7950 1540 60  0001 C CNN
-F 3 "" H 7550 1600 60  0000 C CNN
-	1    7550 1600
-	0    -1   -1   0
-$EndComp
 Wire Wire Line
 	6500 1600 6650 1600
@@
 Wire Wire Line
 	7100 1600 7100 1800
-$Comp
-L modulo_SIM7000G-rescue:1661-conn_ufl-modulo_SIM7000G-rescue J6
-U 1 1 6160E28F
-P 7100 1600
-F 0 "J6" V 7395 1472 60  0000 R CNN
-F 1 "1661" V 7289 1472 60  0000 R CNN
-F 2 "Connector_Coaxial:U.FL_Molex_MCRF_73412-0110_Vertical" H 7500 1540 60  0001 C CNN
-F 3 "" H 7100 1600 60  0000 C CNN
-	1    7100 1600
-	0    -1   -1   0
-$EndComp
-Connection ~ 7100 1600
 $Comp
 L power:+BATT #PWR030
@@
 Wire Wire Line
 	7550 3600 7450 3600
-Text Label 10500 5750 2    50   ~ 0
-NRESET
 Wire Wire Line
 	4750 3500 7000 3500
@@
 Wire Notes Line
 	8400 650  8400 2350
-Text Notes 10300 5500 0    50   ~ 0
-INTERFAZ SERIAL
-Wire Wire Line
-	4050 2800 7550 2800
 Wire Wire Line
 	4050 2800 4050 3150
@@
 	3750 5900 3750 5950
 Wire Wire Line
-	7550 1600 7550 2800
-Wire Wire Line
 	6800 6250 6200 6250
-Text Label 10500 6250 2    50   ~ 0
-POWERKEY
+Wire Wire Line
+	10100 4000 10800 4000
+Wire Wire Line
+	9850 4100 10800 4100
+Wire Wire Line
+	9850 4200 10800 4200
+Wire Wire Line
+	10100 4300 10800 4300
+Text Label 10800 4000 0    50   ~ 0
+DTR
+Text Label 10800 4100 0    50   ~ 0
+RI
+Text Label 10800 4200 0    50   ~ 0
+TX
+Text Label 10800 4300 0    50   ~ 0
+RX
+Wire Wire Line
+	10500 5850 10750 5850
+Text Label 10500 5850 2    50   ~ 0
+RX
+Wire Wire Line
+	10500 5950 10750 5950
+Text Label 10500 5950 2    50   ~ 0
+TX
+Wire Wire Line
+	10500 6050 10750 6050
+Text Label 10500 6050 2    50   ~ 0
+RI
+Wire Wire Line
+	10500 6150 10750 6150
+Text Label 10500 6150 2    50   ~ 0
+DTR
+Wire Wire Line
+	10750 6250 10500 6250
+Wire Wire Line
+	10500 5750 10750 5750
 $Comp
 L Connector_Generic:Conn_01x06 J1
@@
 	1    0    0    -1
 $EndComp
-Wire Wire Line
-	10100 4000 10800 4000
-Wire Wire Line
-	9850 4100 10800 4100
-Wire Wire Line
-	9850 4200 10800 4200
-Wire Wire Line
-	10100 4300 10800 4300
-Wire Wire Line
-	10500 5750 10750 5750
-Wire Wire Line
-	10750 6250 10500 6250
-Text Label 10800 4000 0    50   ~ 0
-DTR
-Text Label 10800 4100 0    50   ~ 0
-RI
-Text Label 10800 4200 0    50   ~ 0
-TX
-Text Label 10800 4300 0    50   ~ 0
-RX
-Text Label 10500 6150 2    50   ~ 0
-DTR
-Wire Wire Line
-	10500 6150 10750 6150
-Text Label 10500 6050 2    50   ~ 0
-RI
-Wire Wire Line
-	10500 6050 10750 6050
-Text Label 10500 5950 2    50   ~ 0
-TX
-Wire Wire Line
-	10500 5950 10750 5950
-Text Label 10500 5850 2    50   ~ 0
-RX
-Wire Wire Line
-	10500 5850 10750 5850
+Text Label 10500 6250 2    50   ~ 0
+POWERKEY
+Text Notes 10300 5500 0    50   ~ 0
+INTERFAZ SERIAL
+Text Label 10500 5750 2    50   ~ 0
+NRESET
+Wire Wire Line
+	4050 2800 7650 2800
+Wire Notes Line
+	6350 700  8100 700
+Wire Notes Line
+	6350 2600 8100 2600
+$Comp
+L Connector:Conn_Coaxial J4
+U 1 1 616C916E
+P 7100 900
+F 0 "J4" V 7000 1050 50  0000 C CNN
+F 1 "GNSS ANT" V 7246 829 50  0000 C CNN
+F 2 "Connector_Coaxial:SMA_Amphenol_132203-12_Horizontal" H 7100 900 50  0001 C CNN
+F 3 " ~" H 7100 900 50  0001 C CNN
+	1    7100 900
+	0    -1   -1   0
+$EndComp
+$Comp
+L Connector:Conn_Coaxial J3
+U 1 1 616936C2
+P 7650 900
+F 0 "J3" V 7550 1050 50  0000 C CNN
+F 1 "RF ANT" V 7796 829 50  0000 C CNN
+F 2 "Connector_Coaxial:SMA_Amphenol_132203-12_Horizontal" H 7650 900 50  0001 C CNN
+F 3 " ~" H 7650 900 50  0001 C CNN
+	1    7650 900
+	0    -1   -1   0
+$EndComp
+Connection ~ 7100 1600
+Text Notes 7750 1450 0    50   ~ 0
+50 Ohms
+Text Notes 7200 1350 0    50   ~ 0
+50 Ohms
+Text Notes 7200 2400 0    50   ~ 0
+50 Ohms
+Wire Notes Line
+	7150 1150 7150 1450
+Wire Notes Line
+	7150 2150 7150 2550
+Wire Notes Line
+	7700 1200 7700 1650
+Wire Wire Line
+	7100 1100 7100 1600
+Wire Wire Line
+	7650 1100 7650 2800
+$Comp
+L power:GND #PWR0106
+U 1 1 6184DB5D
+P 7850 1050
+F 0 "#PWR0106" H 7850 800 50  0001 C CNN
+F 1 "GND" H 7855 877 50  0000 C CNN
+F 2 "" H 7850 1050 50  0001 C CNN
+F 3 "" H 7850 1050 50  0001 C CNN
+	1    7850 1050
+	1    0    0    -1
+$EndComp
+Wire Wire Line
+	7850 1050 7850 900
+$Comp
+L power:GND #PWR0107
+U 1 1 6185E007
+P 7300 1050
+F 0 "#PWR0107" H 7300 800 50  0001 C CNN
+F 1 "GND" H 7305 877 50  0000 C CNN
+F 2 "" H 7300 1050 50  0001 C CNN
+F 3 "" H 7300 1050 50  0001 C CNN
+	1    7300 1050
+	1    0    0    -1
+$EndComp
+Wire Wire Line
+	7300 900  7300 1050
+$Comp
+L Mechanical:Fiducial FID3
+U 1 1 61889E93
+P 9800 1300
+F 0 "FID3" H 9885 1346 50  0000 L CNN
+F 1 "Fiducial" H 9885 1255 50  0000 L CNN
+F 2 "Fiducial:Fiducial_1mm_Mask2mm" H 9800 1300 50  0001 C CNN
+F 3 "~" H 9800 1300 50  0001 C CNN
+	1    9800 1300
+	1    0    0    -1
+$EndComp
 $EndSCHEMATC
