File: pcb/modulo_SIM7000G/_autosave-modulo_SIM7000G.kicad_pcb (KiCad board)
At the start: 2 copper layers, 100 x 60 mm, 58 parts, among them J1 Conector Serial, J2 115Q-BCA0, J5 Jack-DC, J6 1661, J7 1661, Q1 NTE4153NT1G, Q2 NTE4153NT1G, Q3 NTE4153NT1G, U1 SIM7000G, U2 SN74LV1T34DCKR, U3 SN74LV1T34DCKR, U4 SN74LV1T34DCKR, U5 SN74LV1T34DCKR, U6 SN74LV1T34DCKR, U7 MIC29302WU, U8 LM1117-3.3

Commit message: antes de realizar modificaciones rf
Parts:
- moved R12 4.43 mm to (103.0, 114.9), turned to 90 degrees
- moved C13 4.12 mm to (103.0, 108.0), turned to 90 degrees
- moved Q3 3.00 mm to (109.0, 108.0)
Routing:
- net GND: track 599.0 -> 563.4 mm, vias 11 -> 12
- net Net-(C13-Pad1): track 14.1 -> 24.0 mm, vias 0 -> 2
- net +BATT: track 98.5 -> 95.2 mm
- net Net-(Q3-Pad1): track 8.64 -> 11.6 mm
- net Net-(D1-Pad1): track 3.25 -> 5.30 mm
- net Net-(U1-Pad4): track 48.2 -> 47.3 mm
- net Net-(U1-Pad9): track 46.3 -> 47.1 mm
- added copper zone on B.Cu, net GND
Other:
- net class Default: clearance 0.4 -> 0.42; trace_width 0.5 -> 0.45
- rule trace_clearance: 0.4 -> 0.42
- rule trace_min: 0.5 -> 0.4
- board text added: "MODULO 7000 v1.0"
- board text added: "NETLIGHT"
- board text added: "Nota: Grillas utilizadas: 1mm, 0,5 mm . (0,1mm y 0.2mm para alinear componentes)."
