File: pcb/modulo_SIM7000G/modulo_SIM7000G.kicad_pcb (KiCad board)
At the start: 2 copper layers, 100 x 60 mm, 58 parts, among them J1 Conector Serial, J2 115Q-BCA0, J5 Jack-DC, J6 1661, J7 1661, Q1 NTE4153NT1G, Q2 NTE4153NT1G, Q3 NTE4153NT1G, U1 SIM7000G, U2 SN74LV1T34DCKR, U3 SN74LV1T34DCKR, U4 SN74LV1T34DCKR, U5 SN74LV1T34DCKR, U6 SN74LV1T34DCKR, U7 MIC29302WU, U8 LM1117-3.3

Commit message: modificaciones en reglas de diseño del proyecto
Parts:
- moved R12 4.43 mm to (103.0, 114.9), turned to 90 degrees
- moved C13 4.12 mm to (103.0, 108.0), turned to 90 degrees
- moved Q3 3.00 mm to (109.0, 108.0)
Routing:
- net GND: track 599.0 -> 555.2 mm
- net Net-(C13-Pad1): track 14.1 -> 24.0 mm, vias 0 -> 2
- net +BATT: track 98.5 -> 95.2 mm
- net Net-(Q3-Pad1): track 8.64 -> 11.6 mm
- net Net-(D1-Pad1): track 3.25 -> 5.30 mm
- net Net-(U1-Pad4): track 48.2 -> 47.6 mm
Other:
- net class SIM7000 added: clearance 0.4, trace_width 0.5, via_dia 1.4, via_drill 0.7
- net class ci added: clearance 0.1, trace_width 0.4, via_dia 1.4, via_drill 0.7
- rule trace_min: 0.5 -> 0.4
- board text added: "NETLIGHT"

Commit message: antes de realizar modificaciones rf
Routing:
- net GND: track 555.2 -> 563.3 mm, vias 11 -> 12
- net Net-(U1-Pad9): track 46.3 -> 47.1 mm
Other:
- board text added: "MODULO 7000 v1.0"
- board text added: "Nota: Grillas utilizadas: 1mm, 0,5 mm . (0,1mm y 0.2mm para alinear componentes)."
Changed lines of the file:
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@@
   (general
     (thickness 1.6)
-    (drawings 29)
-    (tracks 624)
+    (drawings 31)
+    (tracks 629)
     (zones 0)
     (modules 58)
@@
     (date 2021-09-22)
     (rev "Diego Brengi")
-    (company FIUBA)
-    (comment 1 "Autor: German Velardez")
+    (company "Licencia: CERN Open Hardware Licence Version 2.")
+    (comment 1 "Descripcion. Replica de modulo de comunicacion basado en SIM7000G")
+    (comment 2 "Autor: German Velardez")
   )
   (layers
-    (0 F.Cu signal)
-    (31 B.Cu signal)
+    (0 F.Cu signal hide)
+    (31 B.Cu signal hide)
     (32 B.Adhes user hide)
-    (33 F.Adhes user)
+    (33 F.Adhes user hide)
     (34 B.Paste user hide)
     (35 F.Paste user hide)
@@
   )
   (setup
-    (last_trace_width 0.8)
+    (last_trace_width 0.5)
     (user_trace_width 0.4)
     (user_trace_width 0.5)
@@
     )
   )
+  (gr_text " MODULO 7000 v1.0" (at 90 85) (layer F.SilkS)
+    (effects (font (size 1 1) (thickness 0.15)))
+  )
+  (gr_text "Nota: Grillas utilizadas: 1mm, 0,5 mm .\n(0,1mm y 0.2mm para alinear componentes)." (at 205.5 86) (layer Dwgs.User)
+    (effects (font (size 1 1) (thickness 0.15)))
+  )
   (gr_text NETLIGHT (at 108 112) (layer F.SilkS)
     (effects (font (size 1 1) (thickness 0.25)))
@@
   (segment (start 143 125.5) (end 141.5 127) (width 0.5) (layer F.Cu) (net 1))
   (segment (start 144 125.5) (end 143 125.5) (width 0.5) (layer F.Cu) (net 1))
-  (segment (start 144 124) (end 143.5 123.5) (width 0.5) (layer B.Cu) (net 1))
-  (segment (start 143.5 123.5) (end 144.5 122.5) (width 0.5) (layer B.Cu) (net 1))
   (via (at 144.5 119.5) (size 1.6) (drill 0.8) (layers F.Cu B.Cu) (net 1))
   (segment (start 144.5 122.5) (end 144.5 119.5) (width 0.5) (layer B.Cu) (net 1))
@@
   (segment (start 107.5 108.5) (end 106 107) (width 0.5) (layer F.Cu) (net 1))
   (segment (start 108.35 108.5) (end 107.5 108.5) (width 0.5) (layer F.Cu) (net 1))
+  (segment (start 144 123) (end 145 124) (width 0.5) (layer B.Cu) (net 1))
+  (segment (start 143.5 123.5) (end 144 123) (width 0.5) (layer B.Cu) (net 1))
+  (segment (start 144 123) (end 144.5 122.5) (width 0.5) (layer B.Cu) (net 1))
+  (via (at 149.849972 124.000639) (size 1.6) (drill 0.8) (layers F.Cu B.Cu) (net 1))
+  (segment (start 145.000639 124.000639) (end 149.849972 124.000639) (width 0.5) (layer B.Cu) (net 1))
+  (segment (start 145 124) (end 145.000639 124.000639) (width 0.5) (layer B.Cu) (net 1))
+  (segment (start 151.000639 124.000639) (end 152 125) (width 0.5) (layer F.Cu) (net 1))
+  (segment (start 149.849972 124.000639) (end 151.000639 124.000639) (width 0.5) (layer F.Cu) (net 1))
   (segment (start 104.9625 111) (end 103 109.0375) (width 0.8) (layer F.Cu) (net 2))
   (segment (start 107 111) (end 104.9625 111) (width 0.8) (layer F.Cu) (net 2))
@@
   (segment (start 125 124) (end 125 125.5) (width 0.5) (layer F.Cu) (net 18))
   (segment (start 125 125.5) (end 125 126) (width 0.5) (layer F.Cu) (net 18))
-  (segment (start 125 130.5) (end 125 132.5) (width 0.5) (layer F.Cu) (net 18))
   (via (at 147.5 132) (size 1.4) (drill 0.7) (layers F.Cu B.Cu) (net 18))
-  (segment (start 125 132.5) (end 125 134.5) (width 0.5) (layer F.Cu) (net 18))
-  (via (at 130.5 135) (size 1.4) (drill 0.7) (layers F.Cu B.Cu) (net 18))
-  (segment (start 125.5 135) (end 130.5 135) (width 0.5) (layer F.Cu) (net 18))
-  (segment (start 125 134.5) (end 125.5 135) (width 0.5) (layer F.Cu) (net 18))
-  (segment (start 146 133.5) (end 147.5 132) (width 0.5) (layer B.Cu) (net 18))
-  (segment (start 146 134) (end 146 133.5) (width 0.5) (layer B.Cu) (net 18))
-  (segment (start 145 135) (end 146 134) (width 0.5) (layer B.Cu) (net 18))
-  (segment (start 130.5 135) (end 145 135) (width 0.5) (layer B.Cu) (net 18))
   (segment (start 153.45 128.55) (end 151.949999 130.050001) (width 0.4) (layer F.Cu) (net 18))
   (segment (start 158.4 128.55) (end 153.45 128.55) (width 0.4) (layer F.Cu) (net 18))
   (segment (start 149.449999 130.050001) (end 147.5 132) (width 0.4) (layer F.Cu) (net 18))
   (segment (start 151.949999 130.050001) (end 149.449999 130.050001) (width 0.4) (layer F.Cu) (net 18))
+  (via (at 125 132.5) (size 1.6) (drill 0.8) (layers F.Cu B.Cu) (net 18))
+  (segment (start 125 130.5) (end 125 132.5) (width 0.5) (layer F.Cu) (net 18))
+  (segment (start 146 133.5) (end 147.5 132) (width 0.5) (layer B.Cu) (net 18))
+  (segment (start 146 134) (end 146 133.5) (width 0.5) (layer B.Cu) (net 18))
+  (segment (start 145 135) (end 146 134) (width 0.5) (layer B.Cu) (net 18))
+  (segment (start 126 135) (end 145 135) (width 0.5) (layer B.Cu) (net 18))
+  (segment (start 125 134) (end 126 135) (width 0.5) (layer B.Cu) (net 18))
+  (segment (start 125 132.5) (end 125 134) (width 0.5) (layer B.Cu) (net 18))
   (segment (start 145 132.5) (end 131.5 132.5) (width 0.5) (layer B.Cu) (net 19))
   (segment (start 131.5 132.5) (end 130.5 132.5) (width 0.5) (layer B.Cu) (net 19))
@@
   (segment (start 148.5 128.5) (end 149 128.5) (width 0.5) (layer B.Cu) (net 19))
   (segment (start 148 129) (end 148.5 128.5) (width 0.5) (layer B.Cu) (net 19))
-  (segment (start 147.25 126.75) (end 149 128.5) (width 0.5) (layer F.Cu) (net 19))
-  (segment (start 147.75 124.955998) (end 147.25 125.455998) (width 0.5) (layer F.Cu) (net 19))
-  (segment (start 147.75 123.25) (end 147.75 124.955998) (width 0.5) (layer F.Cu) (net 19))
-  (segment (start 147.25 125.455998) (end 147.25 126.75) (width 0.5) (layer F.Cu) (net 19))
-  (segment (start 148 123) (end 147.75 123.25) (width 0.5) (layer F.Cu) (net 19))
-  (segment (start 156 123) (end 148 123) (width 0.5) (layer F.Cu) (net 19))
-  (segment (start 156.5 123.5) (end 156 123) (width 0.5) (layer F.Cu) (net 19))
-  (segment (start 156.5 123.5) (end 157.324998 123.5) (width 0.5) (layer F.Cu) (net 19))
   (segment (start 157.324998 123.5) (end 158.4 123.5) (width 0.4) (layer F.Cu) (net 19))
+  (segment (start 156.5 123.5) (end 157.324998 123.5) (width 0.5) (layer F.Cu) (net 19))
+  (segment (start 149 122) (end 155 122) (width 0.5) (layer F.Cu) (net 19))
+  (segment (start 147.75 123.25) (end 149 122) (width 0.5) (layer F.Cu) (net 19))
+  (segment (start 155 122) (end 156.5 123.5) (width 0.5) (layer F.Cu) (net 19))
+  (segment (start 147.25 125.455998) (end 147.75 124.955998) (width 0.5) (layer F.Cu) (net 19))
+  (segment (start 147.75 124.955998) (end 147.75 123.25) (width 0.5) (layer F.Cu) (net 19))
+  (segment (start 147.25 126.75) (end 147.25 125.455998) (width 0.5) (layer F.Cu) (net 19))
+  (segment (start 149 128.5) (end 147.25 126.75) (width 0.5) (layer F.Cu) (net 19))
   (segment (start 158.4 118.55) (end 157.85 118) (width 0.5) (layer F.Cu) (net 20))
   (segment (start 149.590002 115.5) (end 148 115.5) (width 0.5) (layer F.Cu) (net 20))

Commit message: termine, falta los modelos 3d de los conectores.
Parts:
- removed J6, J7: 1661, Connector_Coaxial:U.FL_Molex_MCRF_73412-0110_Vertical
- added FID3: Fiducial, Fiducial:Fiducial_1mm_Mask2mm, F.Cu at (167.5, 85.0)
- added J3: RF ANT, Connector_Coaxial:SMA_Amphenol_132203-12_Horizontal, F.Cu at (169.5, 114.0)
- added J4: GNSS ANT, Connector_Coaxial:SMA_Amphenol_132203-12_Horizontal, F.Cu at (169.5, 134.0)
- moved H1 105.2 mm to (171.0, 85.0), turned to 180 degrees
- moved C1 81.9 mm to (171.5, 124.2), turned to 270 degrees
- moved H3 72.5 mm to (98.5, 84.5)
- moved C2 65.1 mm to (165.5, 123.5), turned to 270 degrees
- moved D2 63.6 mm to (169.6, 108.0), turned to 180 degrees
- moved C13 62.2 mm to (160.5, 131.5), turned to 0 degrees
- moved C3 61.5 mm to (163.0, 123.5), turned to 270 degrees
- moved C17 60.6 mm to (160.5, 137.0), turned to 180 degrees
- moved R10 60.5 mm to (136.5, 83.0), turned to 90 degrees
- moved R12 59.2 mm to (160.5, 129.0), turned to 180 degrees
- moved J2 58.7 mm to (106.5, 123.5), turned to 270 degrees
- moved C4 57.9 mm to (160.5, 123.5), turned to 270 degrees
- moved L1 57.3 mm to (160.4, 134.5), turned to 0 degrees
- moved C10 57.0 mm to (116.0, 83.0), turned to 180 degrees
- moved R13 55.9 mm to (163.0, 108.0), turned to 180 degrees
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Routing:
- net GND: track 563.3 -> 259.6 mm, vias 12 -> 13
- net +5VD: track 121.4 -> 42.6 mm
- net Net-(Q1-Pad3): track 49.4 -> 2.85 mm
- net VDD: track 84.6 -> 47.4 mm, vias 4 -> 2
- net /DTR: track 9.64 -> 44.1 mm, vias 0 -> 2
- net Net-(U1-Pad4): track 47.3 -> 14.8 mm
- net Net-(U1-Pad9): track 47.1 -> 20.7 mm
- net Net-(U1-Pad3): track 51.6 -> 25.8 mm, vias 0 -> 1
- net Net-(Q3-Pad1): track 11.6 -> 31.9 mm, vias 0 -> 2
- net Net-(C16-Pad1): track 37.0 -> 17.8 mm
- net +BATT: track 95.2 -> 113.7 mm, vias 2 -> 0
- net Net-(J3-Pad1): track 35.9 -> 17.4 mm
- net Net-(C13-Pad1): track 24.0 -> 5.59 mm, vias 2 -> 0
- net Net-(C15-Pad1): track 35.3 -> 20.1 mm
- net Net-(Q2-Pad3): track 11.1 -> 25.4 mm
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- added copper zone on B.Cu, net GND
Other:
- board size 100 x 60 mm -> 80 x 60 mm
- net class Default: clearance 0.4 -> 0.42; trace_width 0.5 -> 0.45
- net class SIM7000 removed
- net class ci removed
- rule trace_clearance: 0.4 -> 0.42
- board text added: "3.3+"
- board text added: "5+"
- board text added: "ANT GNSS"
- board text added: "ANT RF"
- board text added: "BAT+"
- board text added: "JACK-DC +5"
- board text added: "MODULO SIM7000"
- board text added: "PWKEY"
- board text added: "STATUS"
- board text added: "V1.0"
- board text removed: "3.3V+"
- board text removed: "5V+"
- board text removed: "ANTENA CELULAR"
- board text removed: "ANTENA GNSS"
- board text removed: "INDUSTRIA ARGENTINA"
- board text removed: "LECTOR SIMCARD"
- board text removed: "LED DE ESTADO"
- board text removed: "MODULO 7000 v1.0"
- board text removed: "Nota: Grillas utilizadas: 1mm, 0,5 mm . (0,1mm y 0.2mm para alinear componentes)."
- board text removed: "PKEY"
- board text removed: "VBAT"
